Commit message: Initial commit

File: resources/objects/guitar_new/guitar.urdf (robot description, URDF)
Before this commit: robot guitar.urdf, 1 links, 0 joints
Links:
- link baseLink: geometry collision mesh filename=guitar-wood-10mb.obj scale=0.005 0.005 0.005; visual mesh filename=guitar-wood-10mb.obj scale=0.005 0.005 0.005

File: resources/objects/office_chair/OfficeChair.urdf (robot description, URDF)
Before this commit: robot OfficeChair.urdf, 1 links, 0 joints
Links:
- link baseLink: geometry collision mesh filename=OfficeChair.fbx.obj scale=0.005 0.005 0.005; visual mesh filename=OfficeChair.fbx.obj scale=0.005 0.005 0.005

File: resources/objects/shoes/shoes.urdf (robot description, URDF)
Before this commit: robot shoes.urdf, 1 links, 0 joints
Links:
- link baseLink: geometry collision mesh filename=nb574.obj scale=0.06 0.06 0.06; visual mesh filename=nb574.obj scale=0.06 0.06 0.06
